Commit message: fix: conf for topo
Co-authored-by: BiceMar <bicemarzagora@gmail.com>

File: description/robot_core.xacro (robot description, xacro)
@@ -5,5 +5,5 @@
     <xacro:property name="chassis_width" value="0.250"/>
     <xacro:property name="chassis_height" value="0.120"/>
-    <xacro:property name="chassis_mass" value="1.0"/>
+    <xacro:property name="chassis_mass" value="1.5"/>
     <xacro:property name="wheel_radius" value="0.0725"/>
     <xacro:property name="wheel_thickness" value="0.03"/>
