Commit message: feat: config for MarTopo 🐁
Co-authored-by: BiceMar <bicemarzagora@gmail.com>
Co-authored-by: frovaaa <frovad@usi.ch>

File: description/lidar.xacro (robot description, xacro)
@@ -4,5 +4,5 @@
         <parent link="chassis"/>
         <child link="laser_frame"/>
-        <origin xyz="0.122 0 0.212" rpy="0 0 0"/>
+        <origin xyz="0.360 0.0 0.25" rpy="0 0 3.14"/>
     </joint>
     <link name="laser_frame">

File: description/robot_core.xacro (robot description, xacro)
@@ -2,15 +2,15 @@
 <robot xmlns:xacro="http://www.ros.org/wiki/xacro" >
     <xacro:include filename="inertial_macros.xacro"/>
-    <xacro:property name="chassis_length" value="0.450"/>
-    <xacro:property name="chassis_width" value="0.250"/>
-    <xacro:property name="chassis_height" value="0.120"/>
-    <xacro:property name="chassis_mass" value="1.5"/>
+    <xacro:property name="chassis_length" value="0.470"/>
+    <xacro:property name="chassis_width" value="0.430"/>
+    <xacro:property name="chassis_height" value="0.20"/>
+    <xacro:property name="chassis_mass" value="3.5"/>
     <xacro:property name="wheel_radius" value="0.0725"/>
     <xacro:property name="wheel_thickness" value="0.03"/>
     <xacro:property name="wheel_mass" value="0.05"/>
-    <xacro:property name="wheel_offset_x" value="0.325"/>
+    <xacro:property name="wheel_offset_x" value="0.345"/>
     <xacro:property name="wheel_offset_y" value="0.145"/>
     <xacro:property name="wheel_offset_z" value="0.01"/>
-    <xacro:property name="caster_wheel_radius" value="0.01"/>
+    <xacro:property name="caster_wheel_radius" value="0.015"/>
     <xacro:property name="caster_wheel_mass" value="0.01"/>
     <xacro:property name="caster_wheel_offset_x" value="0.075"/>

File: description/ros2_control.xacro (robot description, xacro)
@@ -11,5 +11,5 @@
                 <param name="baud_rate">57600</param>
                 <param name="timeout_ms">500</param>
-                <param name="enc_counts_per_rev">4480</param>
+                <param name="enc_counts_per_rev">6533</param>
                 <!--param name="enc_counts_per_rev">4480</param-->
             </hardware>
